Commit message: description: RealSense D435i 카메라 프레임 체인 추가 (마운트 나사 구멍 실측 + 인텔 공식 오프셋)
base_link → camera_bottom_screw_frame 실측 x +47.5, y 0, z +48 mm (수평 장착 가정).
그 아래 camera_link(왼쪽 IR, +10.6/+17.5/+12.5mm), camera_depth_frame, camera_color_frame
(+15mm 왼쪽), optical 프레임(rpy -1.5708 0 -1.5708)은 realsense2_description
_d435.urdf.xacro 상수 그대로. 우리 카메라 공장 익스트린식(depth→color 14.9mm)과 일치.
xacro/check_urdf 통과, 합성 변환 확인: RGB 렌즈 (58.1, 32.5, 60.5) mm, optical z 축 = 로봇 앞.
자체 카메라 노드의 frame_id(camera_color_optical_frame)가 TF 트리에 연결됨 → Vision 3D 위치의
base_link 변환 전제. docs/description.md 3.3 절, CLAUDE.md 5·8번, README 갱신.

Co-Authored-By: Claude Fable 5.1 <noreply@anthropic.com>

File: description/urdf/turtlebot3_burger.urdf (robot description, URDF)
Before this commit: robot turtlebot3_burger, 7 links, 6 joints
Links:
- added link ${namespace}camera_bottom_screw_frame
- added link ${namespace}camera_color_frame
- added link ${namespace}camera_color_optical_frame
- added link ${namespace}camera_depth_frame
- added link ${namespace}camera_depth_optical_frame
- added link ${namespace}camera_link, mass 0.072; visual box size=0.02505 0.090 0.025
Joints:
- added joint ${namespace}camera_color_joint: type fixed, parent ${namespace}camera_link, child ${namespace}camera_color_frame, origin xyz=0 0.015 0 rpy=0 0 0
- added joint ${namespace}camera_color_optical_joint: type fixed, parent ${namespace}camera_color_frame, child ${namespace}camera_color_optical_frame, origin xyz=0 0 0 rpy=-1.5708 0 -1.5708
- added joint ${namespace}camera_depth_joint: type fixed, parent ${namespace}camera_link, child ${namespace}camera_depth_frame, origin xyz=0 0 0 rpy=0 0 0
- added joint ${namespace}camera_depth_optical_joint: type fixed, parent ${namespace}camera_depth_frame, child ${namespace}camera_depth_optical_frame, origin xyz=0 0 0 rpy=-1.5708 0 -1.5708
- added joint ${namespace}camera_link_joint: type fixed, parent ${namespace}camera_bottom_screw_frame, child ${namespace}camera_link, origin xyz=0.0106 0.0175 0.0125 rpy=0 0 0
- added joint ${namespace}camera_mount_joint: type fixed, parent ${namespace}base_link, child ${namespace}camera_bottom_screw_frame, origin xyz=0.0475 0 0.048 rpy=0 0 0

Commit message: 실측 반영: IMU 위치(OpenCR 보드 중심 -0.030,0,0.060) + Nav2 실측 footprint + 카메라 수평 확인
- URDF imu_joint xyz -0.032,0,0.068 → -0.030,0,0.060 (보드 기하학적 중심 실측, 2026-09-08;
  IMU 칩이 아닌 보드 중심이지만 이 로봇 속도에선 EKF 에 무의미한 차이). 카메라 기울기 실측
  수평 → pitch 0 확정.
- nav2_params.yaml: local/global costmap 의 robot_radius 0.105(표준 임시) →
  footprint "[[0.062,0.09],[-0.22,0.09],[-0.22,-0.09],[0.062,-0.09]]" (앞 = 카메라 전면
  0.0475+0.0149, 뒤 -0.220, 좌우 ±0.090 실측). 전장 28cm 로 원 하나로는 뒤쪽이 잘렸음.
- docs: description.md(표·3.2·검증·다음), my_navigation.md(4장·표·8장), CLAUDE.md 5·8번.
  URDF YAML/xacro/check_urdf, nav2 YAML 검증 통과.

Co-Authored-By: Claude Fable 5.1 <noreply@anthropic.com>

File: description/urdf/turtlebot3_burger.urdf (robot description, URDF)
Before this commit: robot turtlebot3_burger, 13 links, 12 joints
Joints:
- joint ${namespace}imu_joint: origin xyz=-0.032 0 0.068 rpy=0 0 -1.57 -> xyz=-0.030 0 0.060 rpy=0 0 -1.57

Commit message: description: RViz 로봇 모델을 실물 CAD 통짜 메시로 교체 + my_description 패키지화
- 사용자가 실물을 CAD 로 그린 STL(원점 base_link, m 단위, 바퀴·LDS·카메라 포함)을
  Open3D quadric decimation 으로 118만→10만 삼각형(59MB→5MB) 경량화해 커밋
  (원본 my_turtleBot3_burger.stl 은 .gitignore)
- URDF: base_link visual → package://my_description/meshes/my_turtlebot3_burger_lowpoly.stl,
  바퀴·base_scan·camera_link 의 개별 visual 제거 (링크·조인트·TF 는 그대로)
- description/ 을 ament 패키지 my_description 으로 (package.xml, CMakeLists: urdf·meshes 설치),
  docker-compose 에서 ./description → /overlay_ws/src/my_description 중첩 마운트
- 컨테이너에서 robot_state_publisher + RViz 로 검증: 메시 로드, 폭·앞은 실측 footprint 와 일치,
  뒤쪽 55mm 차이(footprint -0.220 vs CAD -0.165)는 확인 필요 항목으로 기록
- docs: description.md 3.4 절·검증 기록, server_setup(마운트·빌드·source 주의), pi_setup(메시 불필요),
  README/CLAUDE 구조, docs/images/robot_model_cad.png

Co-Authored-By: Claude Fable 5.1 <noreply@anthropic.com>

File: description/urdf/turtlebot3_burger.urdf (robot description, URDF)
Before this commit: robot turtlebot3_burger, 13 links, 12 joints
Links:
- link ${namespace}base_link: geometry collision box size=0.140 0.140 0.143; visual mesh filename=package://my_description/meshes/my_turtlebot3_burger_lowpol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 scale=1 1 1
- link ${namespace}base_scan: geometry collision cylinder length=0.0315 radius=0.055
- link ${namespace}camera_link: geometry 
- link ${namespace}wheel_left_link: geometry collision cylinder length=0.018 radius=0.033
- link ${namespace}wheel_right_link: geometry collision cylinder length=0.018 radius=0.033
